File: Shortcut-3000.kicad_sch (KiCad schematic)
At the start: 33 parts, among them SW1 SW_Push, SW10 SW_Push, SW11 SW_Push, SW12 SW_Push, SW13 SW_Push, SW14 SW_Push, SW15 SW_Push, SW16 RotaryEncoder_Switch, SW17 RotaryEncoder_Switch, SW2 SW_Push, SW3 SW_Push, SW4 SW_Push, SW5 SW_Push, SW6 SW_Push, SW7 SW_Push, SW8 SW_Push, SW9 SW_Push

Commit message: Add 12 magnetic I2C connectors and pull-ups to schematic
J1-J12 use the female magnetic pogo connector with pinout
1=GND 2=SCL 3=+3V3 4=SDA 5=GND. I2C1 runs from Pico GP14 (SDA) and
GP15 (SCL) with 4.7k pull-ups (R1, R2) to +3V3. The Pico 3V3 pin
now drives the +3V3 net instead of being marked no-connect. Sheet
enlarged to A3 to make room.

Co-Authored-By: Claude Opus 5.5 <noreply@anthropic.com>
Claude-Session: https://claude.ai/code/session_01YbA9Kuqksf6ZcSb59HLVep
Parts:
- added J1, J10, J11, J12, J2, J3, J4, J5, J6, J7, J8, J9: MagneticPogo_1x05_Female, Shortcut-3000:MagneticPogo_1x05_P2.54mm_Female, symbol Shortcut-3000:MagneticPogo_1x05_Female
- added R1, R2: 4.7k, Resistor_THT:R_Axial_DIN0207_L6.3mm_D2.5mm_P7.62mm_Horizontal, symbol Device:R
Connections:
- net GND: now also J1.1 (Pin_1), J1.5 (Pin_5), J10.1 (Pin_1), J10.5 (Pin_5), J11.1 (Pin_1), J11.5 (Pin_5), J12.1 (Pin_1), J12.5 (Pin_5), J2.1 (Pin_1), J2.5 (Pin_5), J3.1 (Pin_1), J3.5 (Pin_5), J4.1 (Pin_1), J4.5 (Pin_5), J5.1 (Pin_1), J5.5 (Pin_5), J6.1 (Pin_1), J6.5 (Pin_5), J7.1 (Pin_1), J7.5 (Pin_5), J8.1 (Pin_1), J8.5 (Pin_5), J9.1 (Pin_1), J9.5 (Pin_5)
- net SDA: now reaches A1.19 (GPIO14)
- net SDA: now also J1.4 (Pin_4), J10.4 (Pin_4), J11.4 (Pin_4), J12.4 (Pin_4), J2.4 (Pin_4), J3.4 (Pin_4), J4.4 (Pin_4), J5.4 (Pin_4), J6.4 (Pin_4), J7.4 (Pin_4), J8.4 (Pin_4), J9.4 (Pin_4), R1.2
- net SCL: now reaches A1.20 (GPIO15)
- net SCL: now also J1.2 (Pin_2), J10.2 (Pin_2), J11.2 (Pin_2), J12.2 (Pin_2), J2.2 (Pin_2), J3.2 (Pin_2), J4.2 (Pin_2), J5.2 (Pin_2), J6.2 (Pin_2), J7.2 (Pin_2), J8.2 (Pin_2), J9.2 (Pin_2), R2.2
- net +3V3: now reaches A1.36 (3V3)
- net +3V3: now also J1.3 (Pin_3), J10.3 (Pin_3), J11.3 (Pin_3), J12.3 (Pin_3), J2.3 (Pin_3), J3.3 (Pin_3), J4.3 (Pin_3), J5.3 (Pin_3), J6.3 (Pin_3), J7.3 (Pin_3), J8.3 (Pin_3), J9.3 (Pin_3), R1.1, R2.1
- no-connect marks 17 -> 16
Other:
- note added: "Magnetic connectors J1-J12: 1=GND 2=SCL 3=+3V3 4=SDA 5=GND I2C1 on Pico: GP14 = SDA, GP15 = SCL, 4.7k pull-ups R1/R2 to +3V3"
