File: Shortcut-3000.kicad_sch (KiCad schematic)
At the start: 47 parts, among them J1 MagneticPogo_1x05_Female, J10 MagneticPogo_1x05_Female, J11 MagneticPogo_1x05_Female, J12 MagneticPogo_1x05_Female, J2 MagneticPogo_1x05_Female, J3 MagneticPogo_1x05_Female, J4 MagneticPogo_1x05_Female, J5 MagneticPogo_1x05_Female, J6 MagneticPogo_1x05_Female, J7 MagneticPogo_1x05_Female, J8 MagneticPogo_1x05_Female, J9 MagneticPogo_1x05_Female, U1 TCA9548APWR, U2 TCA9548APWR

Commit message: Update PCB layout and schematic
Parts:
- added R33, R34, R35, R36, R37, R38, R39, R40, R41, R42: 10k, Resistor_SMD:R_0805_2012Metric, symbol Device:R
Connections:
- net +3V3: now also R33.1, R34.1, R35.1, R36.1, R37.1, R38.1, R39.1, R40.1, R41.1, R42.1
- net INT_J6: now reaches A1.10 (GP13)
- net INT_J6: now also J6.5 (Pin_5), R37.2
- net INT_J5: now reaches A1.11 (GP12)
- net INT_J5: now also J5.5 (Pin_5), R36.2
- net INT_J1: now reaches A1.13 (GP10)
- net INT_J1: now also J1.5 (Pin_5), R33.2
- net INT_J4: now reaches A1.21 (GP2)
- net INT_J4: now also J4.5 (Pin_5), R35.2
- net INT_J8: now reaches A1.4 (GP29)
- net INT_J8: now also J8.5 (Pin_5), R38.2
- net INT_J12: now reaches A1.5 (GP28)
- net INT_J12: now also J12.5 (Pin_5), R42.2
- net INT_J9: now reaches A1.6 (GP27)
- net INT_J9: now also J9.5 (Pin_5), R39.2
- net INT_J10: now reaches A1.7 (GP26)
- net INT_J10: now also J10.5 (Pin_5), R40.2
- net INT_J11: now reaches A1.8 (GP15)
- net INT_J11: now also J11.5 (Pin_5), R41.2
- net INT_J7: now reaches A1.9 (GP14)
- net INT_J7: now also J7.5 (Pin_5), R6.2
- removed net INT0: A1.15 (GP8), J1.5 (Pin_5), J2.5 (Pin_5), J3.5 (Pin_5), J4.5 (Pin_5), J5.5 (Pin_5), J6.5 (Pin_5), R5.2
- removed net INT1: A1.14 (GP9), J10.5 (Pin_5), J11.5 (Pin_5), J12.5 (Pin_5), J7.5 (Pin_5), J8.5 (Pin_5), J9.5 (Pin_5), R6.2
- new net INT_J2: A1.14 (GP9), J2.5 (Pin_5), R34.2
- new net INT_J3: A1.15 (GP8), J3.5 (Pin_5), R5.2
Other:
- note added: "Magnetic connectors J1-J12 (4 x 3 module grid, 25.4 mm pitch): 1=GND 2=SCL 3=+3V3 4=SDA 5=INT (open-drain, active low) Bus 0: GP4 = SDA0, GP5 = SCL0 -> U1 TCA9548A; J1-J6 on U1 channels 0-5 Bus 1: GP6 = SDA1, GP7 = SCL1 -> U2 TCA9548A; J7-J12 on U2 channels 0-5 INT: one line per slot, INT_J1-INT_J12 -> GP10=J1, GP9=J2, GP8=J3, GP2=J4, GP12=J5, GP13=J6, GP14=J7, GP29=J8, GP27=J9, GP26=J10, GP15=J1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"
- note removed: "Magnetic connectors J1-J12 (4 x 3 module grid, 25.4 mm pitch): 1=GND 2=SCL 3=+3V3 4=SDA 5=INT (open-drain, active low) Bus 0: GP4 = SDA0, GP5 = SCL0 -> U1 TCA9548A; J1-J6 on U1 channels 0-5; GP8 = INT0 (shared by J1-J6) Bus 1: GP6 = SDA1, GP7 = SCL1 -> U2 TCA9548A; J7-J12 on U2 channels 0-5; GP9 = INT1 (shared by J7-J12) Pull-ups to +3V3: R1-R4 4.7k on SDA0/SCL0/SDA1/SCL1, R5-R6 10k on INT, R7-R8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"
