File: Shortcut-3000.kicad_pcb (KiCad board)
At the start: 2 copper layers, 105.5 x 82.5 mm, 47 parts, among them J1 MagneticPogo_1x05_Female, J10 MagneticPogo_1x05_Female, J11 MagneticPogo_1x05_Female, J12 MagneticPogo_1x05_Female, J2 MagneticPogo_1x05_Female, J3 MagneticPogo_1x05_Female, J4 MagneticPogo_1x05_Female, J5 MagneticPogo_1x05_Female, J6 MagneticPogo_1x05_Female, J7 MagneticPogo_1x05_Female, J8 MagneticPogo_1x05_Female, J9 MagneticPogo_1x05_Female, U1 TCA9548APWR, U2 TCA9548APWR

Commit message: Update PCB layout and schematic
Parts:
- added R33: 10k, Resistor_SMD:R_0805_2012Metric, B.Cu at (142.5, 52.9)
- added R34: 10k, Resistor_SMD:R_0805_2012Metric, B.Cu at (167.9, 52.9)
- added R35: 10k, Resistor_SMD:R_0805_2012Metric, B.Cu at (218.7, 50.9)
- added R36: 10k, Resistor_SMD:R_0805_2012Metric, B.Cu at (142.5, 78.3)
- added R37: 10k, Resistor_SMD:R_0805_2012Metric, B.Cu at (167.9, 78.3)
- added R38: 10k, Resistor_SMD:R_0805_2012Metric, B.Cu at (213.7, 80.3)
- added R39: 10k, Resistor_SMD:R_0805_2012Metric, B.Cu at (142.5, 103.7)
- added R40: 10k, Resistor_SMD:R_0805_2012Metric, B.Cu at (167.9, 103.7)
- added R41: 10k, Resistor_SMD:R_0805_2012Metric, B.Cu at (193.3, 103.7)
- added R42: 10k, Resistor_SMD:R_0805_2012Metric, B.Cu at (214.2, 105.5)
- moved R5 4.65 mm to (194.8, 53.8), turned to 0 degrees
Connections:
- A1 pad 10: unconnected-(A1-GP13-Pad10) -> /INT_J6
- A1 pad 11: unconnected-(A1-GP12-Pad11) -> /INT_J5
- A1 pad 13: unconnected-(A1-GP10-Pad13) -> /INT_J1
- A1 pad 14: /INT1 -> /INT_J2
- A1 pad 15: /INT0 -> /INT_J3
- A1 pad 21: unconnected-(A1-GP2-Pad21) -> /INT_J4
- A1 pad 4: unconnected-(A1-GP29-Pad4) -> /INT_J8
- A1 pad 5: unconnected-(A1-GP28-Pad5) -> /INT_J12
- A1 pad 6: unconnected-(A1-GP27-Pad6) -> /INT_J9
- A1 pad 7: unconnected-(A1-GP26-Pad7) -> /INT_J10
- A1 pad 8: unconnected-(A1-GP15-Pad8) -> /INT_J11
- A1 pad 9: unconnected-(A1-GP14-Pad9) -> /INT_J7
- J1 pad 5: /INT0 -> /INT_J1
- J10 pad 5: /INT1 -> /INT_J10
- J11 pad 5: /INT1 -> /INT_J11
- J12 pad 5: /INT1 -> /INT_J12
- J2 pad 5: /INT0 -> /INT_J2
- J3 pad 5: /INT0 -> /INT_J3
- J4 pad 5: /INT0 -> /INT_J4
- J5 pad 5: /INT0 -> /INT_J5
- J6 pad 5: /INT0 -> /INT_J6
- J7 pad 5: /INT1 -> /INT_J7
- J8 pad 5: /INT1 -> /INT_J8
- J9 pad 5: /INT1 -> /INT_J9
- R5 pad 2: /INT0 -> /INT_J3
- R6 pad 2: /INT1 -> /INT_J7
Routing:
- net GND: track 347.0 -> 38.3 mm, vias 6 -> 9
- net /INT1: track 172.8 -> 0.00 mm
- net /INT0: track 149.0 -> 0.00 mm, vias 2 -> 0
- net /INT_J11: track 0.00 -> 102.5 mm
- net /INT_J9: track 0.00 -> 87.6 mm, vias 0 -> 2
- net /INT_J1: track 0.00 -> 71.2 mm, vias 0 -> 4
- net /INT_J5: track 0.00 -> 69.2 mm, vias 0 -> 2
- net /INT_J10: track 0.00 -> 61.6 mm, vias 0 -> 2
- net /INT_J2: track 0.00 -> 47.7 mm, vias 0 -> 2
- net /INT_J6: track 0.00 -> 43.8 mm, vias 0 -> 2
- net /INT_J12: track 0.00 -> 32.4 mm, vias 0 -> 1
- net /INT_J7: track 0.00 -> 21.1 mm, vias 0 -> 1
- net /INT_J3: track 0.00 -> 12.5 mm, vias 0 -> 2
- net /INT_J4: track 0.00 -> 7.82 mm
- net /INT_J8: track 0.00 -> 6.37 mm
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- added copper zone on F.Cu, net GND
